Commit message: FEAT: add mapping.launch modify robot urdf

File: src/my_robot/urdf/my_robot.xacro (robot description, xacro)
@@ -148,33 +148,40 @@
   </gazebo>
   <link name="camera">
-    <inertial>
-      <mass value="0.1"/>
-      <origin value="0 0 0"/>
-      <inertia
-        ixx="1e-6" ixy="0" ixz="0"
-        iyy="1e-6" iyz="0"
-        izz="1e-6"
-        />
-    </inertial>
-    <collision name="camera_collision">
-      <origin xyz="0 0 0" rpy="0 0 0"/>
-      <geometry>
-        <box size=".05 .05 .05"/>
-      </geometry>
-    </collision>
-    <visual name="camera_visual">
-      <origin xyz="0 0 0" rpy="0 0 0"/>
-      <geometry>
-        <box size=".05 .05 .05"/>
-      </geometry>
-      <material name="green"/>
-    </visual>
+      <inertial>
+          <mass value="0.1"/>
+          <origin value="0 0 0"/>
+          <inertia
+              ixx="1e-6" ixy="0" ixz="0"
+              iyy="1e-6" iyz="0"
+              izz="1e-6"
+              />
+      </inertial>
+      <collision name="camera_collision">
+          <origin xyz="0 0 0" rpy="0 0 0"/>
+          <geometry>
+              <box size=".05 .05 .05"/>
+          </geometry>
+      </collision>
+      <visual name="camera_visual">
+          <origin xyz="0 0 0" rpy="0 0 0"/>
+          <geometry>
+              <box size=".05 .05 .05"/>
+          </geometry>
+          <material name="green"/>
+      </visual>
   </link>
   <joint type="fixed" name="camera_joint">
-    <origin xyz=".2 0 0" rpy="0 0 0"/>
-    <child link="camera"/>
-    <parent link="chassis"/>
-    <axis xyz="0 1 0" rpy="0 0 0"/>
-  </joint>
+      <origin xyz=".2 0 0" rpy="0 0 0"/>
+      <child link="camera"/>
+      <parent link="chassis"/>
+      <axis xyz="0 1 0" rpy="0 0 0"/>
+  </joint>
+  <joint name="camera_optical_joint" type="fixed">
+    <origin xyz="0 0 0" rpy="-1.5707 0 -1.5707"/>
+    <parent link="camera"/>
+    <child link="camera_link_optical"/>
+  </joint>
+  <link name="camera_link_optical">
+  </link>
   <link name="hokuyo">
     <inertial>

Commit message: adding mapping launch file and upgrade sensor

File: src/my_robot/urdf/my_robot.xacro (robot description, xacro)
@@ -180,7 +180,7 @@
     <origin xyz="0 0 0" rpy="-1.5707 0 -1.5707"/>
     <parent link="camera"/>
-    <child link="camera_link_optical"/>
-  </joint>
-  <link name="camera_link_optical">
+    <child link="optical"/>
+  </joint>
+  <link name="optical">
   </link>
   <link name="hokuyo">
